File: kicad/veloce.kicad_pcb (KiCad board)
At the start: 2 copper layers, 100 x 100 mm, 95 parts, among them J1 OUT, J10 BAT, J11 HVBin, J12 HVBout, J13 LVBin, J14 LVBout, J15 5Vout, J16 Brake, J17 USB_A_stacked, J18 USB_C_Receptacle_USB2.0, J19 USB_C_Receptacle_USB2.0, J2 OUT, J20 Inputs, J3 OUT, J4 OUT, J5 OUT, J6 OUT, J7 OUT, J8 OUT, J9 BAT, P1 CONN_1, P10 CONN_1, P11 CONN_1, P12 CONN_1, P13 CONN_1, P14 CONN_1, P15 CONN_1, P16 CONN_1, P2 CONN_1, P3 CONN_1, P4 CONN_1, P5 CONN_1, P6 CONN_1, P7 CONN_1, P8 CONN_1, P9 CONN_1, Q1 IRLR7843TRPBF, Q2 IRLR7843TRPBF, Q3 AO3400A, Q4 AO3400A, Q5 AO3400A, Q6 AO3400A, Q7 AO3400A, Q8 AO3400A, U1 Adafruit_HUZZAH_ESP32_breakou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

Commit message: prototype gerber ready
Parts:
- removed P1, P10, P11, P12, P13, P14, P15, P16, P2, P3, P4, P5, P6, P7, P8, P9: CONN_1, veloce:TestPoint_THTPad_D2.0mm_Drill1.0mm
- J10, J9: value BAT -> PWR
- J11: value HVBin -> PWR
- J12: value HVBout -> PWR
- J13: value LVBin -> PWR
- J14: value LVBout -> PWR
- J15: value 5Vout -> PWR
- U1: footprint veloce:Adafruit_HUZZAH_ESP32_breakout -> veloce:Adafruit_HUZZAH_ESP32_breakout_sparepads
Connections:
- net Net-(D1-Pad2) renamed /OP1
- net Net-(D2-Pad2) renamed /OP2
- net Net-(D3-Pad2) renamed /OP3
- net Net-(D4-Pad2) renamed /OP4
- net Net-(D5-Pad2) renamed /OP5
- net Net-(D6-Pad2) renamed /OP6
- net Net-(D7-Pad2) renamed /OP7
- net Net-(D8-Pad2) renamed /OP8
- J10 pad 2: /GND -> /12V
- J11 pad 1: /72V -> /12V
- J11 pad 2: /GND -> /5V
- J12 pad 1: /12V -> /5V
- J13 pad 1: /12V -> /GND
- J14 pad 1: /5V -> /GND
- J15 pad 1: /5V -> /GND
- J16 pad 1: /BRAKE -> /GND
- J16 pad 2: /GND -> /BRAKE
- J9 pad 2: /GND -> /72V
Routing:
- net /GND: track 0.00 -> 566.6 mm, vias 0 -> 8
- net /12V: track 0.00 -> 277.0 mm
- net /5V: track 0.00 -> 189.4 mm
- net /3V3: track 0.00 -> 136.3 mm
- net /BRAKE: track 0.00 -> 53.6 mm
- net /IN8: track 0.00 -> 51.1 mm
- net /IN1: track 0.00 -> 49.7 mm
- net /OUT8: track 0.00 -> 49.5 mm
- net /IN7: track 0.00 -> 43.7 mm
- net /OUT1: track 0.00 -> 42.3 mm
- net /OUT7: track 0.00 -> 41.6 mm
- net /IN2: track 0.00 -> 40.7 mm
- net /OUT2: track 0.00 -> 39.2 mm
- net /IN6: track 0.00 -> 37.3 mm
- net /OUT6: track 0.00 -> 33.5 mm
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- added copper zone on B.Cu, net /12V
- added copper zone on B.Cu, net /GND
- added copper zone on B.Cu, net /OP1
- added copper zone on F.Cu, net /OP1
- added copper zone on B.Cu, net /OP2
- added copper zone on F.Cu, net /OP2
Other:
- outline, holes or cut-outs redrawn
- net class 0.50mm added: clearance 0.2, trace_width 0.5, via_dia 0.8, via_drill 0.4
- net class 1.00mm added: clearance 0.2, trace_width 1, via_dia 0.8, via_drill 0.4
- net class 1.50mm added: clearance 0.2, trace_width 1.5, via_dia 0.8, via_drill 0.4
- net class 2.00mm added: clearance 0.2, trace_width 2, via_dia 0.8, via_drill 0.4

Commit message: added superawesome logos
Parts:
- added G1: Logo_Veloce, veloce:VR_logo, F.Cu at (179.5, 131.0)
- added G2: Logo_Veloce, veloce:VR_logo1, F.Cu at (179.5, 131.0)
- added G3: Logo_Veloce, veloce:VR_logo2, B.Cu at (170.0, 126.0)
- added G4: Logo_Veloce, veloce:VR_logo3, B.Cu at (170.0, 126.0)

Commit message: added labels and right angle connector 3D models
Parts:
- removed J10, J11, J12, J13, J14, J15: PWR, veloce:TerminalBlock_Wurth_1377-2_Horizontal
- removed J16: Brake, veloce:TerminalBlock_Wurth_1377-2_Horizontal
- added kibuzzard-614E1815: G***, label, B.Cu at (151.0, 68.0)
- added kibuzzard-614E1883: G***, label, B.Cu at (151.0, 78.0)
- added kibuzzard-614E188E: G***, label, B.Cu at (151.0, 88.0)
- added kibuzzard-614E1899: G***, label, B.Cu at (151.0, 98.0)
- added kibuzzard-614E18A2: G***, label, B.Cu at (151.0, 108.0)
- added kibuzzard-614E18AA: G***, label, B.Cu at (151.0, 118.0)
- added kibuzzard-614E18B2: G***, label, B.Cu at (151.0, 128.0)
- added kibuzzard-614E18BA: G***, label, B.Cu at (151.0, 138.0)
- added kibuzzard-614E196C: G***, label, B.Cu at (232.0, 68.0)
- added kibuzzard-614E19A5: G***, label, B.Cu at (232.0, 78.0)
- added kibuzzard-614E19AF: G***, label, B.Cu at (232.0, 88.0)
- added kibuzzard-614E19B6: G***, label, B.Cu at (232.0, 98.0)
- added kibuzzard-614E19C0: G***, label, B.Cu at (232.0, 108.0)
- added kibuzzard-614E19C8: G***, label, B.Cu at (232.0, 118.0)
- added kibuzzard-614E19D4: G***, label, B.Cu at (232.0, 128.0)
- added kibuzzard-614E19DD: G***, label, B.Cu at (232.0, 138.0)
- added kibuzzard-614E1BE6: G***, label, B.Cu at (198.5, 129.0)
- added kibuzzard-614E1BE6: G***, label, F.Cu at (199.5, 135.0)
- added kibuzzard-614E1CD8: G***, label, B.Cu at (198.5, 133.5)
- added kibuzzard-614E1CD8: G***, label, F.Cu at (199.5, 139.5)
- added kibuzzard-614E1DC4: G***, label, B.Cu at (171.0, 146.0)
- added kibuzzard-614E1DE5: G***, label, B.Cu at (158.5, 146.0)
- added kibuzzard-614E1E36: G***, label, B.Cu at (181.0, 146.0)
- added kibuzzard-614E1E6D: G***, label, B.Cu at (203.5, 146.0)
- added kibuzzard-614E1E9D: G***, label, B.Cu at (226.0, 146.0)
- G1: footprint veloce:VR_logo -> veloce:VR_logo4
- G2: footprint veloce:VR_logo1 -> veloce:VR_logo5
- J9: footprint veloce:TerminalBlock_Wurth_1377-2_Horizontal -> veloce:TerminalBlock_Wurth_1377-16_Horizontal
- R17, R18, R19, R20, R21, R22, R23, R24, R25, R26, R27, R28, R29: footprint veloce:R_Axial_DIN0207_L6.3mm_D2.5mm_P7.62mm_Horizontal -> veloce:r_0805_THT
- moved R21 3.81 mm to (224.8, 140.5)
- moved R22 3.81 mm to (224.8, 65.5)
- moved R23 3.81 mm to (224.8, 75.5)
- moved R24 3.81 mm to (224.8, 85.5)
- moved R25 3.81 mm to (224.8, 95.5)
- moved R26 3.81 mm to (224.8, 105.5)
- moved R27 3.81 mm to (224.8, 115.5)
- moved R28 3.81 mm to (224.8, 125.5)
- moved R29 3.81 mm to (224.8, 135.5)
- moved R17 3.79 mm to (200.3, 68.0)
- moved R18 3.79 mm to (200.3, 71.0)
- moved R19 3.79 mm to (211.3, 68.0)
- moved R20 3.79 mm to (211.3, 71.0)
- moved G1 3.35 mm to (181.0, 134.0)
- moved G2 3.35 mm to (181.0, 134.0)
Routing:
- net /3V3: track 136.3 -> 124.7 mm
- net /5V: track 189.4 -> 201.0 mm
- net /GND: track 566.6 -> 578.2 mm
- net /IN2: track 40.7 -> 45.3 mm
- net /BRAKE: track 53.6 -> 58.1 mm
- net /IN7: track 43.7 -> 48.0 mm
- net /IN8: track 51.1 -> 55.3 mm
- net /IN3: track 33.5 -> 37.7 mm
- net /IN6: track 37.3 -> 40.6 mm
- net Net-(J19-PadB5): track 20.9 -> 23.8 mm
- net Net-(J18-PadB5): track 20.6 -> 23.5 mm
- net Net-(JP9-Pad2): track 0.00 -> 2.86 mm
- net Net-(JP8-Pad2): track 0.00 -> 2.86 mm
- net Net-(JP7-Pad2): track 0.00 -> 2.86 mm
- net Net-(JP6-Pad2): track 0.00 -> 2.86 mm
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Other:
- board text added: "AND THUS WE GET THE OUTPUTS HERE - TWO ARE JUICY, OTHERS NOT."
- board text added: "BRAINZ"
- board text added: "HERE BE THE INPUTS - ALL EIGHT OF 'EM"
- board text added: "HERE COMES THE POWER - FLIP BOARD TO SEE WHAT GOES WHERE"

Commit message: JLCpcb production files ready
Parts:
- removed the kibuzzard-614E188E at (151.0, 88.0)
- removed the kibuzzard-614E18AA at (151.0, 118.0)
- removed the kibuzzard-614E18BA at (151.0, 138.0)
- removed the kibuzzard-614E196C at (232.0, 68.0)
- removed the kibuzzard-614E19AF at (232.0, 88.0)
- removed the kibuzzard-614E19DD at (232.0, 138.0)
- removed the kibuzzard-614E1BE6 at (198.5, 129.0)
- removed the kibuzzard-614E1BE6 at (199.5, 135.0)
- removed the kibuzzard-614E1CD8 at (198.5, 133.5)
- removed the kibuzzard-614E1CD8 at (199.5, 139.5)
- removed the kibuzzard-614E1E6D at (203.5, 146.0)
- removed the kibuzzard-614E1E9D at (226.0, 146.0)
- added G5: LOGO_WL, veloce:logo_butterfly_silk_15x12, B.Cu at (205.0, 74.0)
- added G6: LOGO_WL, veloce:logo_butterfly_mask_15x12, B.Cu at (205.0, 74.0)
- added G7: Logo_OSHW, veloce:Logo_OSHW-11.4x12mm_SilkScreen, B.Cu at (200.0, 110.0)
- added G8: Logo_Wyolum, veloce:logo_wyolum_silk_20x8, B.Cu at (184.0, 75.0)
- added G9: Logo_Wyolum, veloce:logo_wyolum_mask_20x8, B.Cu at (184.0, 75.0)
- added kibuzzard-614E188E: #G12, veloce:label_OUT3, B.Cu at (150.5, 88.0)
- added kibuzzard-614E18AA: #G15, veloce:label_OUT6, B.Cu at (150.5, 118.0)
- added kibuzzard-614E18BA: #G17, veloce:label_OUT8, B.Cu at (150.5, 138.0)
- added kibuzzard-614E196C: #G18, veloce:label_IN1, B.Cu at (232.0, 68.0)
- added kibuzzard-614E19AF: #G20, veloce:label_IN3, B.Cu at (232.0, 88.0)
- added kibuzzard-614E19DD: #G25, veloce:label_IN8, B.Cu at (232.0, 138.0)
- added kibuzzard-614E1BE6: #G3, veloce:label_Cafe_Veloce, B.Cu at (202.5, 129.0)
- added kibuzzard-614E1BE6: #G1, veloce:label_Cafe_Veloce, F.Cu at (199.5, 135.5)
- added kibuzzard-614E1CD8: #G4, veloce:label_VeloRaptor, B.Cu at (202.5, 133.5)
- added kibuzzard-614E1CD8: #G2, veloce:label_VeloRaptor, F.Cu at (199.5, 140.0)
- added kibuzzard-614E1E6D: #G8, veloce:label_GND, B.Cu at (204.0, 146.0)
- added kibuzzard-614E1E9D: #G9, veloce:label_Brake, B.Cu at (226.0, 146.0)
- kibuzzard-614E1815: value G*** -> #G10; footprint label -> veloce:label_OUT1
- kibuzzard-614E1883: value G*** -> #G11; footprint label -> veloce:label_OUT2
- kibuzzard-614E1899: value G*** -> #G13; footprint label -> veloce:label_OUT4
- kibuzzard-614E18A2: value G*** -> #G14; footprint label -> veloce:label_OUT5
- kibuzzard-614E18B2: value G*** -> #G16; footprint label -> veloce:label_OUT7
- kibuzzard-614E19A5: value G*** -> #G19; footprint label -> veloce:label_IN2
- kibuzzard-614E19B6: value G*** -> #G21; footprint label -> veloce:label_IN4
- kibuzzard-614E19C0: value G*** -> #G22; footprint label -> veloce:label_IN5
- kibuzzard-614E19C8: value G*** -> #G23; footprint label -> veloce:label_IN6
- kibuzzard-614E19D4: value G*** -> #G24; footprint label -> veloce:label_IN7
- kibuzzard-614E1DC4: value G*** -> #G6; footprint label -> veloce:label_12V
- kibuzzard-614E1DE5: value G*** -> #G5; footprint label -> veloce:label_72V
- kibuzzard-614E1E36: value G*** -> #G7; footprint label -> veloce:label_5V
- moved kibuzzard-614E1815 0.50 mm to (150.5, 68.0)
- moved kibuzzard-614E1883 0.50 mm to (150.5, 78.0)
- moved kibuzzard-614E1899 0.50 mm to (150.5, 98.0)
- moved kibuzzard-614E18A2 0.50 mm to (150.5, 108.0)
- moved kibuzzard-614E18B2 0.50 mm to (150.5, 128.0)
- turned R11 to 0 degrees
- turned R12 to 0 degrees
- turned R15 to 0 degrees
- turned R16 to 0 degrees
- turned R21 to 0 degrees
- turned R22 to 0 degrees
- turned R24 to 0 degrees
- turned R26 to 0 degrees
- turned R28 to 0 degrees
- turned R3 to 0 degrees
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Connections:
- R11 pad 1: /OUT5 -> /GND
- R11 pad 2: /GND -> /OUT5
- R12 pad 1: /OUT6 -> /GND
- R12 pad 2: /GND -> /OUT6
- R15 pad 1: /OUT7 -> /GND
- R15 pad 2: /GND -> /OUT7
- R16 pad 1: /OUT8 -> /GND
- R16 pad 2: /GND -> /OUT8
- R21 pad 1: /BRAKE -> Net-(JP1-Pad2)
- R21 pad 2: Net-(JP1-Pad2) -> /BRAKE
- R22 pad 1: /IN1 -> Net-(JP2-Pad2)
- R22 pad 2: Net-(JP2-Pad2) -> /IN1
- R24 pad 1: /IN3 -> Net-(JP4-Pad2)
- R24 pad 2: Net-(JP4-Pad2) -> /IN3
- R26 pad 1: /IN5 -> Net-(JP6-Pad2)
- R26 pad 2: Net-(JP6-Pad2) -> /IN5
- R28 pad 1: /IN7 -> Net-(JP8-Pad2)
- R28 pad 2: Net-(JP8-Pad2) -> /IN7
- R3 pad 1: /OUT1 -> /GND
- R3 pad 2: /GND -> /OUT1
- R4 pad 1: /OUT2 -> /GND
- R4 pad 2: /GND -> /OUT2
- R7 pad 1: /OUT3 -> /GND
- R7 pad 2: /GND -> /OUT3
- R8 pad 1: /OUT4 -> /GND
- R8 pad 2: /GND -> /OUT4
Routing:
- net /IN3: track 37.7 -> 38.8 mm
- net /IN1: track 50.3 -> 51.1 mm
