File: kicad/veloce.sch (KiCad schematic (older format))
At the start: 95 parts, among them J1 OUT, J10 BAT, J11 HVBin, J12 HVBout, J13 LVBin, J14 LVBout, J15 5Vout, J16 Brake, J17 USB_A_stacked, J18 USB_C_Receptacle_USB2.0, J19 USB_C_Receptacle_USB2.0, J2 OUT, J20 Inputs, J3 OUT, J4 OUT, J5 OUT, J6 OUT, J7 OUT, J8 OUT, J9 BAT, P1 CONN_1, P10 CONN_1, P11 CONN_1, P12 CONN_1, P13 CONN_1, P14 CONN_1, P15 CONN_1, P16 CONN_1, P2 CONN_1, P3 CONN_1, P4 CONN_1, P5 CONN_1, P6 CONN_1, P7 CONN_1, P8 CONN_1, P9 CONN_1, Q1 IRLR7843TRPBF, Q2 IRLR7843TRPBF, Q3 AO3400A, Q4 AO3400A, Q5 AO3400A, Q6 AO3400A, Q7 AO3400A, Q8 AO3400A, U1 Adafruit_HUZZAH_ESP32_breakou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

Commit message: prototype gerber ready
Parts:
- removed P1, P10, P11, P12, P13, P14, P15, P16, P2, P3, P4, P5, P6, P7, P8, P9: CONN_1, veloce:TestPoint_THTPad_D2.0mm_Drill1.0mm, symbol veloce:CONN_1
- J10, J9: value BAT -> PWR; Field4 [+] -> (none); Field5 [-] -> (none)
- J11: value HVBin -> PWR; Field4 [+] -> (none); Field5 [-] -> (none)
- J12: value HVBout -> PWR; Field4 [+] -> (none); Field5 [-] -> (none)
- J13: value LVBin -> PWR; Field4 [+] -> (none); Field5 [-] -> (none)
- J14: value LVBout -> PWR; Field4 [+] -> (none); Field5 [-] -> (none)
- J15: value 5Vout -> PWR; Field4 [+] -> (none); Field5 [-] -> (none)
- J16: Field4 [+] -> (none); Field5 [-] -> (none)
- U1: footprint veloce:Adafruit_HUZZAH_ESP32_breakout -> veloce:Adafruit_HUZZAH_ESP32_breakout_sparepads
Connections:
- net labels added: OP1, OP2, OP3, OP4, OP5, OP6, OP7, OP8
- wire segments 262 -> 300
- no-connect marks 16 -> 46
Other:
- note added: "NOTE :\nThis block allows setting\neach input with pull up\nor pull down"
- note removed: "NOTE :\nThis block allows setting each input \nwith pull up or pull down resistor"
- moved on the sheet: J10, J11, J12, J13, J14, J15, J16, J17A, J17B, J18, J19, J20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

Commit message: added superawesome logos
Parts:
- added G1: Logo_Veloce, veloce:VR_logo, symbol veloce:Logo_Veloce
- added G2: Logo_Veloce, veloce:VR_logo1, symbol veloce:Logo_Veloce
- added G3: Logo_Veloce, veloce:VR_logo2, symbol veloce:Logo_Veloce
- added G4: Logo_Veloce, veloce:VR_logo3, symbol veloce:Logo_Veloce
Other:
- moved on the sheet: H1, H2, H3, H4
Changed lines of the file:
@@
 L Mechanical:MountingHole H1
 U 1 1 6154A6B7
-P 9300 6225
-F 0 "H1" H 9300 6100 50  0000 C CNN
-F 1 "Screw" H 9300 6025 50  0000 C CNN
-F 2 "veloce:MountingHole_3.2mm_M3_Pad_Via" H 9300 6225 50  0001 C CNN
-F 3 "~" H 9300 6225 50  0001 C CNN
-	1    9300 6225
+P 7975 6225
+F 0 "H1" H 7975 6100 50  0000 C CNN
+F 1 "Screw" H 7975 6025 50  0000 C CNN
+F 2 "veloce:MountingHole_3.2mm_M3_Pad_Via" H 7975 6225 50  0001 C CNN
+F 3 "~" H 7975 6225 50  0001 C CNN
+	1    7975 6225
 	1    0    0    -1
 $EndComp
@@
 L Mechanical:MountingHole H2
 U 1 1 6154B1BE
-P 9600 6225
-F 0 "H2" H 9600 6100 50  0000 C CNN
-F 1 "Screw" H 9600 6025 50  0000 C CNN
-F 2 "veloce:MountingHole_3.2mm_M3_Pad_Via" H 9600 6225 50  0001 C CNN
-F 3 "~" H 9600 6225 50  0001 C CNN
-	1    9600 6225
+P 8275 6225
+F 0 "H2" H 8275 6100 50  0000 C CNN
+F 1 "Screw" H 8275 6025 50  0000 C CNN
+F 2 "veloce:MountingHole_3.2mm_M3_Pad_Via" H 8275 6225 50  0001 C CNN
+F 3 "~" H 8275 6225 50  0001 C CNN
+	1    8275 6225
 	1    0    0    -1
 $EndComp
@@
 L Mechanical:MountingHole H3
 U 1 1 6154B340
-P 9900 6225
-F 0 "H3" H 9900 6100 50  0000 C CNN
-F 1 "Screw" H 9900 6025 50  0000 C CNN
-F 2 "veloce:MountingHole_3.2mm_M3_Pad_Via" H 9900 6225 50  0001 C CNN
-F 3 "~" H 9900 6225 50  0001 C CNN
-	1    9900 6225
+P 8575 6225
+F 0 "H3" H 8575 6100 50  0000 C CNN
+F 1 "Screw" H 8575 6025 50  0000 C CNN
+F 2 "veloce:MountingHole_3.2mm_M3_Pad_Via" H 8575 6225 50  0001 C CNN
+F 3 "~" H 8575 6225 50  0001 C CNN
+	1    8575 6225
 	1    0    0    -1
 $EndComp
@@
 L Mechanical:MountingHole H4
 U 1 1 6154B4D2
-P 10200 6225
-F 0 "H4" H 10200 6100 50  0000 C CNN
-F 1 "Screw" H 10200 6025 50  0000 C CNN
-F 2 "veloce:MountingHole_3.2mm_M3_Pad_Via" H 10200 6225 50  0001 C CNN
-F 3 "~" H 10200 6225 50  0001 C CNN
-	1    10200 6225
+P 8875 6225
+F 0 "H4" H 8875 6100 50  0000 C CNN
+F 1 "Screw" H 8875 6025 50  0000 C CNN
+F 2 "veloce:MountingHole_3.2mm_M3_Pad_Via" H 8875 6225 50  0001 C CNN
+F 3 "~" H 8875 6225 50  0001 C CNN
+	1    8875 6225
 	1    0    0    -1
 $EndComp
@@
 Text Label 10400 5075 0    30   ~ 0
 OP8
+$Comp
+L veloce:Logo_Veloce G2
+U 1 1 6157474A
+P 8975 6850
+F 0 "G2" H 8975 6525 60  0001 C CNN
+F 1 "Logo_Veloce" H 8975 7175 60  0001 C CNN
+F 2 "veloce:VR_logo1" H 8975 6850 50  0001 C CNN
+F 3 "" H 8975 6850 50  0001 C CNN
+	1    8975 6850
+	1    0    0    -1
+$EndComp
+$Comp
+L veloce:Logo_Veloce G3
+U 1 1 61576B43
+P 8975 6850
+F 0 "G3" H 8975 6525 60  0001 C CNN
+F 1 "Logo_Veloce" H 8975 7175 60  0001 C CNN
+F 2 "veloce:VR_logo2" H 8975 6850 50  0001 C CNN
+F 3 "" H 8975 6850 50  0001 C CNN
+	1    8975 6850
+	1    0    0    -1
+$EndComp
+$Comp
+L veloce:Logo_Veloce G4
+U 1 1 61579302
+P 8975 6850
+F 0 "G4" H 8975 6525 60  0001 C CNN
+F 1 "Logo_Veloce" H 8975 7175 60  0001 C CNN
+F 2 "veloce:VR_logo3" H 8975 6850 50  0001 C CNN
+F 3 "" H 8975 6850 50  0001 C CNN
+	1    8975 6850
+	1    0    0    -1
+$EndComp
+$Comp
+L veloce:Logo_Veloce G1
+U 1 1 6157F0FB
+P 8975 6850
+F 0 "G1" H 8975 6525 60  0001 C CNN
+F 1 "Logo_Veloce" H 8975 7175 60  0001 C CNN
+F 2 "veloce:VR_logo" H 8975 6850 50  0001 C CNN
+F 3 "" H 8975 6850 50  0001 C CNN
+	1    8975 6850
+	1    0    0    -1
+$EndComp
 $EndSCHEMATC

Commit message: added labels and right angle connector 3D models
Parts:
- removed J10, J11, J12, J13, J14, J15: PWR, veloce:TerminalBlock_Wurth_1377-2_Horizontal, symbol veloce:Screw_Terminal_01x02
- removed J16: Brake, veloce:TerminalBlock_Wurth_1377-2_Horizontal, symbol veloce:Screw_Terminal_01x02
- G1: footprint veloce:VR_logo -> veloce:VR_logo4
- G2: footprint veloce:VR_logo1 -> veloce:VR_logo5
- J9: footprint veloce:TerminalBlock_Wurth_1377-2_Horizontal -> veloce:TerminalBlock_Wurth_1377-16_Horizontal; symbol veloce:Screw_Terminal_01x02 -> veloce:Screw_Terminal_01x16
- R17, R18, R19, R20, R21, R22, R23, R24, R25, R26, R27, R28, R29: footprint veloce:R_Axial_DIN0207_L6.3mm_D2.5mm_P7.62mm_Horizontal -> veloce:r_0805_THT
Connections:
- net 12V: now also J9.4 (Pin_4), J9.5 (Pin_5)
- net 5V: now also J9.6 (Pin_6), J9.7 (Pin_7)
- net 72V: now also J9.3 (Pin_3)
- net BRAKE: now also J9.16 (Pin_16)
- net GND: now also J9.10 (Pin_10), J9.11 (Pin_11), J9.12 (Pin_12), J9.13 (Pin_13), J9.14 (Pin_14), J9.15 (Pin_15), J9.8 (Pin_8), J9.9 (Pin_9)
Other:
- note added: "BRAKE"
Changed lines of the file:
@@
 GND
 $Comp
-L veloce:Screw_Terminal_01x02 J9
+L veloce:Screw_Terminal_01x16 J9
 U 1 1 617B0E01
-P 2775 700
-F 0 "J9" H 2850 700 50  0000 L CNB
-F 1 "PWR" H 2975 600 40  0001 L CNN
-F 2 "veloce:TerminalBlock_Wurth_1377-2_Horizontal" H 2775 700 50  0001 C CNN
-F 3 "https://www.we-online.de/katalog/datasheet/691137710002.pdf" H 2775 700 50  0001 C CNN
-F 4 "691137710002" H 2775 700 50  0001 C CNN "PN"
-	1    2775 700
-	-1   0    0    -1
-$EndComp
-$Comp
-L veloce:Screw_Terminal_01x02 J10
-U 1 1 617D3132
-P 2775 900
-F 0 "J10" H 2850 900 50  0000 L CNB
-F 1 "PWR" H 2975 800 40  0001 L CNN
-F 2 "veloce:TerminalBlock_Wurth_1377-2_Horizontal" H 2775 900 50  0001 C CNN
-F 3 "~" H 2775 900 50  0001 C CNN
-	1    2775 900
-	-1   0    0    -1
-$EndComp
-$Comp
-L veloce:Screw_Terminal_01x02 J16
-U 1 1 614A67B5
-P 2775 2100
-F 0 "J16" H 2850 2100 50  0000 L CNB
-F 1 "Brake" H 3275 2025 40  0000 L CNN
-F 2 "veloce:TerminalBlock_Wurth_1377-2_Horizontal" H 2775 2100 50  0001 C CNN
-F 3 "~" H 2775 2100 50  0001 C CNN
-	1    2775 2100
-	-1   0    0    -1
-$EndComp
-$Comp
-L veloce:Screw_Terminal_01x02 J15
-U 1 1 614A5EE9
-P 2775 1900
-F 0 "J15" H 2850 1900 50  0000 L CNB
-F 1 "PWR" H 2975 1800 40  0001 L CNN
-F 2 "veloce:TerminalBlock_Wurth_1377-2_Horizontal" H 2775 1900 50  0001 C CNN
-F 3 "~" H 2775 1900 50  0001 C CNN
-	1    2775 1900
+P 2775 1400
+F 0 "J9" H 2850 2175 50  0000 L CNB
+F 1 "PWR" H 2975 1300 40  0001 L CNN
+F 2 "veloce:TerminalBlock_Wurth_1377-16_Horizontal" H 2775 1400 50  0001 C CNN
+F 3 "https://www.we-online.de/katalog/datasheet/691137710002.pdf" H 2775 1400 50  0001 C CNN
+F 4 "691137710002" H 2775 1400 50  0001 C CNN "PN"
+	1    2775 1400
 	-1   0    0    -1
 $EndComp
@@
 $EndComp
 $Comp
-L veloce:Screw_Terminal_01x02 J14
-U 1 1 61B0998B
-P 2775 1700
-F 0 "J14" H 2850 1700 50  0000 L CNB
-F 1 "PWR" H 2975 1600 40  0001 L CNN
-F 2 "veloce:TerminalBlock_Wurth_1377-2_Horizontal" H 2775 1700 50  0001 C CNN
-F 3 "~" H 2775 1700 50  0001 C CNN
-	1    2775 1700
-	-1   0    0    -1
-$EndComp
-$Comp
-L veloce:Screw_Terminal_01x02 J13
-U 1 1 617E33B9
-P 2775 1500
-F 0 "J13" H 2850 1500 50  0000 L CNB
-F 1 "PWR" H 2975 1400 40  0001 L CNN
-F 2 "veloce:TerminalBlock_Wurth_1377-2_Horizontal" H 2775 1500 50  0001 C CNN
-F 3 "~" H 2775 1500 50  0001 C CNN
-	1    2775 1500
-	-1   0    0    -1
-$EndComp
-$Comp
-L veloce:Screw_Terminal_01x02 J12
-U 1 1 617E2E21
-P 2775 1300
-F 0 "J12" H 2850 1300 50  0000 L CNB
-F 1 "PWR" H 2975 1200 40  0001 L CNN
-F 2 "veloce:TerminalBlock_Wurth_1377-2_Horizontal" H 2775 1300 50  0001 C CNN
-F 3 "~" H 2775 1300 50  0001 C CNN
-	1    2775 1300
-	-1   0    0    -1
-$EndComp
-$Comp
-L veloce:Screw_Terminal_01x02 J11
-U 1 1 617D342A
-P 2775 1100
-F 0 "J11" H 2850 1100 50  0000 L CNB
-F 1 "PWR" H 2975 1000 40  0001 L CNN
-F 2 "veloce:TerminalBlock_Wurth_1377-2_Horizontal" H 2775 1100 50  0001 C CNN
-F 3 "~" H 2775 1100 50  0001 C CNN
-	1    2775 1100
-	-1   0    0    -1
-$EndComp
-$Comp
 L veloce:R R20
 U 1 1 61673E32
@@
 F 0 "R20" V 5950 6000 50  0000 L CNB
 F 1 "22k" V 5850 6000 40  0000 L CNN
-F 2 "veloce:R_Axial_DIN0207_L6.3mm_D2.5mm_P7.62mm_Horizontal" V 5780 6075 50  0001 C CNN
+F 2 "veloce:r_0805_THT" V 5780 6075 50  0001 C CNN
 F 3 "~" H 5850 6075 50  0001 C CNN
 	1    5850 6075
@@
 F 0 "R19" V 5750 6000 50  0000 L CNB
 F 1 "22k" V 5650 6000 40  0000 L CNN
-F 2 "veloce:R_Axial_DIN0207_L6.3mm_D2.5mm_P7.62mm_Horizontal" V 5580 6075 50  0001 C CNN
+F 2 "veloce:r_0805_THT" V 5580 6075 50  0001 C CNN
 F 3 "~" H 5650 6075 50  0001 C CNN
 	1    5650 6075
@@
 F 0 "R18" V 4225 6000 50  0000 L CNB
 F 1 "22k" V 4125 6000 40  0000 L CNN
-F 2 "veloce:R_Axial_DIN0207_L6.3mm_D2.5mm_P7.62mm_Horizontal" V 4055 6075 50  0001 C CNN
+F 2 "veloce:r_0805_THT" V 4055 6075 50  0001 C CNN
 F 3 "~" H 4125 6075 50  0001 C CNN
 	1    4125 6075
@@
 F 0 "R17" V 4025 6000 50  0000 L CNB
 F 1 "22k" V 3925 6000 40  0000 L CNN
-F 2 "veloce:R_Axial_DIN0207_L6.3mm_D2.5mm_P7.62mm_Horizontal" V 3855 6075 50  0001 C CNN
+F 2 "veloce:r_0805_THT" V 3855 6075 50  0001 C CNN
 F 3 "~" H 3925 6075 50  0001 C CNN
 	1    3925 6075
@@
 F 0 "R21" V 3100 4175 50  0000 L CNB
 F 1 "10k" V 3200 4175 40  0000 L CNN
-F 2 "veloce:R_Axial_DIN0207_L6.3mm_D2.5mm_P7.62mm_Horizontal" V 3130 4250 50  0001 C CNN
+F 2 "veloce:r_0805_THT" V 3130 4250 50  0001 C CNN
 F 3 "~" H 3200 4250 50  0001 C CNN
 	1    3200 4250
@@
 F 0 "R22" V 5075 1600 50  0000 L CNB
 F 1 "10k" V 5175 1600 40  0000 L CNN
-F 2 "veloce:R_Axial_DIN0207_L6.3mm_D2.5mm_P7.62mm_Horizontal" V 5105 1675 50  0001 C CNN
+F 2 "veloce:r_0805_THT" V 5105 1675 50  0001 C CNN
 F 3 "~" H 5175 1675 50  0001 C CNN
 	1    5175 1675
@@
 F 0 "R23" V 6425 1600 50  0000 L CNB
 F 1 "10k" V 6525 1600 40  0000 L CNN
-F 2 "veloce:R_Axial_DIN0207_L6.3mm_D2.5mm_P7.62mm_Horizontal" V 6455 1675 50  0001 C CNN
+F 2 "veloce:r_0805_THT" V 6455 1675 50  0001 C CNN
 F 3 "~" H 6525 1675 50  0001 C CNN
 	1    6525 1675
@@
 F 0 "R24" V 5075 2200 50  0000 L CNB
 F 1 "10k" V 5175 2200 40  0000 L CNN
-F 2 "veloce:R_Axial_DIN0207_L6.3mm_D2.5mm_P7.62mm_Horizontal" V 5105 2275 50  0001 C CNN
+F 2 "veloce:r_0805_THT" V 5105 2275 50  0001 C CNN
 F 3 "~" H 5175 2275 50  0001 C CNN
 	1    5175 2275
@@
 F 0 "R25" V 6425 2200 50  0000 L CNB
 F 1 "10k" V 6525 2200 40  0000 L CNN
-F 2 "veloce:R_Axial_DIN0207_L6.3mm_D2.5mm_P7.62mm_Horizontal" V 6455 2275 50  0001 C CNN
+F 2 "veloce:r_0805_THT" V 6455 2275 50  0001 C CNN
 F 3 "~" H 6525 2275 50  0001 C CNN
 	1    6525 2275
@@
 F 0 "R27" V 6425 2800 50  0000 L CNB
 F 1 "10k" V 6525 2800 40  0000 L CNN
-F 2 "veloce:R_Axial_DIN0207_L6.3mm_D2.5mm_P7.62mm_Horizontal" V 6455 2875 50  0001 C CNN
+F 2 "veloce:r_0805_THT" V 6455 2875 50  0001 C CNN
 F 3 "~" H 6525 2875 50  0001 C CNN
 	1    6525 2875
@@
 F 0 "R26" V 5075 2800 50  0000 L CNB
 F 1 "10k" V 5175 2800 40  0000 L CNN
-F 2 "veloce:R_Axial_DIN0207_L6.3mm_D2.5mm_P7.62mm_Horizontal" V 5105 2875 50  0001 C CNN
+F 2 "veloce:r_0805_THT" V 5105 2875 50  0001 C CNN
 F 3 "~" H 5175 2875 50  0001 C CNN
 	1    5175 2875
@@
 F 0 "R28" V 5075 3400 50  0000 L CNB
 F 1 "10k" V 5175 3400 40  0000 L CNN
-F 2 "veloce:R_Axial_DIN0207_L6.3mm_D2.5mm_P7.62mm_Horizontal" V 5105 3475 50  0001 C CNN
+F 2 "veloce:r_0805_THT" V 5105 3475 50  0001 C CNN
 F 3 "~" H 5175 3475 50  0001 C CNN
 	1    5175 3475
@@
 F 0 "R29" V 6425 3400 50  0000 L CNB
 F 1 "10k" V 6525 3400 40  0000 L CNN
-F 2 "veloce:R_Axial_DIN0207_L6.3mm_D2.5mm_P7.62mm_Horizontal" V 6455 3475 50  0001 C CNN
+F 2 "veloce:r_0805_THT" V 6455 3475 50  0001 C CNN
 F 3 "~" H 6525 3475 50  0001 C CNN
 	1    6525 3475
@@
 F 0 "G2" H 8975 6525 60  0001 C CNN
 F 1 "Logo_Veloce" H 8975 7175 60  0001 C CNN
-F 2 "veloce:VR_logo1" H 8975 6850 50  0001 C CNN
+F 2 "veloce:VR_logo5" H 8975 6850 50  0001 C CNN
 F 3 "" H 8975 6850 50  0001 C CNN
 	1    8975 6850
@@
 F 0 "G1" H 8975 6525 60  0001 C CNN
 F 1 "Logo_Veloce" H 8975 7175 60  0001 C CNN
-F 2 "veloce:VR_logo" H 8975 6850 50  0001 C CNN
+F 2 "veloce:VR_logo4" H 8975 6850 50  0001 C CNN
 F 3 "" H 8975 6850 50  0001 C CNN
 	1    8975 6850
 	1    0    0    -1
 $EndComp
+Text Notes 2075 2200 0    40   ~ 0
+BRAKE
 $EndSCHEMATC

Commit message: JLCpcb production files ready
Parts:
- added G5: LOGO_WL, veloce:logo_butterfly_silk_15x12, symbol veloce:LOGO_WL
- added G6: LOGO_WL, veloce:logo_butterfly_mask_15x12, symbol veloce:LOGO_WL
- added G7: Logo_OSHW, veloce:Logo_OSHW-11.4x12mm_SilkScreen, symbol veloce:Logo_OSHW
- added G8: Logo_Wyolum, veloce:logo_wyolum_silk_20x8, symbol veloce:Logo_Wyolum
- added G9: Logo_Wyolum, veloce:logo_wyolum_mask_20x8, symbol veloce:Logo_Wyolum
Connections:
- net BRAKE: now also R21.2; no longer R21.1
- net GND: now also R11.1, R12.1, R15.1, R16.1, R3.1, R4.1, R7.1, R8.1; no longer R11.2, R12.2, R15.2, R16.2, R3.2, R4.2, R7.2, R8.2
- net IN1: now also R22.2; no longer R22.1
- net IN3: now also R24.2; no longer R24.1
- net IN5: now also R26.2; no longer R26.1
- net IN7: now also R28.2; no longer R28.1
- net OUT1: now also R3.2; no longer R3.1
- net OUT2: now also R4.2; no longer R4.1
- net OUT3: now also R7.2; no longer R7.1
- net OUT4: now also R8.2; no longer R8.1
- net OUT5: now also R11.2; no longer R11.1
- net OUT6: now also R12.2; no longer R12.1
- net OUT7: now also R15.2; no longer R15.1
- net OUT8: now also R16.2; no longer R16.1
- net at JP1.2 (C): now also R21.1; no longer R21.2
- net at JP2.2 (C): now also R22.1; no longer R22.2
- net at JP4.2 (C): now also R24.1; no longer R24.2
- net at JP6.2 (C): now also R26.1; no longer R26.2
- net at JP8.2 (C): now also R28.1; no longer R28.2
Changed lines of the file:
@@
 F 3 "~" H 9700 5525 50  0001 C CNN
 	1    9700 5525
-	1    0    0    -1
+	-1   0    0    1
 $EndComp
 $Comp
@@
 F 3 "~" H 9700 4175 50  0001 C CNN
 	1    9700 4175
-	1    0    0    -1
+	-1   0    0    1
 $EndComp
 $Comp
@@
 F 3 "~" H 9700 2825 50  0001 C CNN
 	1    9700 2825
-	1    0    0    -1
+	-1   0    0    1
 $EndComp
 $Comp
@@
 F 3 "~" H 9700 1475 50  0001 C CNN
 	1    9700 1475
-	1    0    0    -1
+	-1   0    0    1
 $EndComp
 $Comp
@@
 F 3 "~" H 7550 5525 50  0001 C CNN
 	1    7550 5525
-	1    0    0    -1
+	-1   0    0    1
 $EndComp
 $Comp
@@
 F 3 "~" H 7550 4175 50  0001 C CNN
 	1    7550 4175
-	1    0    0    -1
+	-1   0    0    1
 $EndComp
 $Comp
@@
 F 3 "~" H 7550 2825 50  0001 C CNN
 	1    7550 2825
-	1    0    0    -1
+	-1   0    0    1
 $EndComp
 $Comp
@@
 F 3 "~" H 7550 1475 50  0001 C CNN
 	1    7550 1475
-	1    0    0    -1
+	-1   0    0    1
 $EndComp
 $Comp
@@
 F 3 "~" H 3200 4250 50  0001 C CNN
 	1    3200 4250
-	0    -1   -1   0
+	0    1    1    0
 $EndComp
 Text Label 3500 4550 2    40   ~ 0
@@
 F 3 "~" H 5175 1675 50  0001 C CNN
 	1    5175 1675
-	0    -1   -1   0
+	0    1    1    0
 $EndComp
 $Comp
@@
 F 3 "~" H 5175 2275 50  0001 C CNN
 	1    5175 2275
-	0    -1   -1   0
+	0    1    1    0
 $EndComp
 $Comp
@@
 F 3 "~" H 5175 2875 50  0001 C CNN
 	1    5175 2875
-	0    -1   -1   0
+	0    1    1    0
 $EndComp
 $Comp
@@
 F 3 "~" H 5175 3475 50  0001 C CNN
 	1    5175 3475
-	0    -1   -1   0
+	0    1    1    0
 $EndComp
 $Comp
@@
 Text Notes 2075 2200 0    40   ~ 0
 BRAKE
+$Comp
+L veloce:Logo_OSHW G7
+U 1 1 616DFC4B
+P 10800 7000
+F 0 "G7" H 10800 6950 40  0001 C CNN
+F 1 "Logo_OSHW" H 10800 7100 40  0001 C CNN
+F 2 "veloce:Logo_OSHW-11.4x12mm_SilkScreen" H 10800 7000 60  0001 C CNN
+F 3 "" H 10800 7000 60  0000 C CNN
+	1    10800 7000
+	1    0    0    -1
+$EndComp
+$Comp
+L veloce:LOGO_WL G5
+U 1 1 616EBDBF
+P 7900 6700
+F 0 "G5" H 7900 6564 60  0001 C CNN
+F 1 "LOGO_WL" H 7900 6836 60  0001 C CNN
+F 2 "veloce:logo_butterfly_silk_15x12" H 7900 6700 60  0001 C CNN
+F 3 "" H 7900 6700 60  0001 C CNN
+	1    7900 6700
+	1    0    0    -1
+$EndComp
+$Comp
+L veloce:LOGO_WL G6
+U 1 1 6151078E
+P 7900 6700
+F 0 "G6" H 7900 6564 60  0001 C CNN
+F 1 "LOGO_WL" H 7900 6836 60  0001 C CNN
+F 2 "veloce:logo_butterfly_mask_15x12" H 7900 6700 60  0001 C CNN
+F 3 "" H 7900 6700 60  0001 C CNN
+	1    7900 6700
+	1    0    0    -1
+$EndComp
+$Comp
+L veloce:Logo_Wyolum G8
+U 1 1 6154CB45
+P 7275 6675
+F 0 "G8" H 7275 6585 60  0001 C CNN
+F 1 "Logo_Wyolum" H 7275 6765 60  0001 C CNN
+F 2 "veloce:logo_wyolum_silk_20x8" H 7275 6675 50  0001 C CNN
+F 3 "" H 7275 6675 50  0001 C CNN
+	1    7275 6675
+	1    0    0    -1
+$EndComp
+$Comp
+L veloce:Logo_Wyolum G9
+U 1 1 61594C76
+P 7275 6675
+F 0 "G9" H 7275 6585 60  0001 C CNN
+F 1 "Logo_Wyolum" H 7275 6765 60  0001 C CNN
+F 2 "veloce:logo_wyolum_mask_20x8" H 7275 6675 50  0001 C CNN
+F 3 "" H 7275 6675 50  0001 C CNN
+	1    7275 6675
+	1    0    0    -1
+$EndComp
 $EndSCHEMATC
