File: kicad_v2/MOSFETS.sch (KiCad schematic (older format))
At the start: 72 parts, among them J1 OUT, J2 OUT, J3 OUT, J4 OUT, J5 OUT, J6 OUT, J7 OUT, J8 OUT, Q1 FQD11P06TM, Q10 RYM002N05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

Commit message: JLCpcb production files ready for CV rev 2
Parts:
- D1, D2, D3, D4, D5, D6, D7, D8: footprint veloce:D_SMB -> veloce:D_SMA
- Q10, Q12, Q14, Q16, Q2, Q4, Q6, Q8: value RYM002N05 -> RUM001L02T2CL
Changed lines of the file:
@@
 F 0 "D1" V 3875 975 50  0000 R CNB
 F 1 "B220A-13-F" H 3925 1050 30  0000 R CNN
-F 2 "veloce:D_SMB" V 3800 975 50  0001 C CNN
+F 2 "veloce:D_SMA" V 3800 975 50  0001 C CNN
 F 3 "~" V 3800 975 50  0001 C CNN
 	1    3800 975
@@
 AR Path="/6276F530/627E9C4D" Ref="Q2"  Part="1"
 F 0 "Q2" H 3275 1800 50  0000 L CNB
-F 1 "RYM002N05" V 3350 1400 30  0000 L CNN
+F 1 "RUM001L02T2CL" V 3350 1400 30  0000 L CNN
 F 2 "veloce:SOT-723" H 3350 1625 29  0001 L CNN
 F 3 "" H 3150 1675 60  0000 C CNN
@@
 F 0 "D2" V 3875 2725 50  0000 R CNB
 F 1 "B220A-13-F" H 3925 2800 30  0000 R CNN
-F 2 "veloce:D_SMB" V 3800 2725 50  0001 C CNN
+F 2 "veloce:D_SMA" V 3800 2725 50  0001 C CNN
 F 3 "~" V 3800 2725 50  0001 C CNN
 	1    3800 2725
@@
 AR Path="/6276F530/627E9CA2" Ref="Q4"  Part="1"
 F 0 "Q4" H 3275 3550 50  0000 L CNB
-F 1 "RYM002N05" V 3350 3150 30  0000 L CNN
+F 1 "RUM001L02T2CL" V 3350 3150 30  0000 L CNN
 F 2 "veloce:SOT-723" H 3350 3375 29  0001 L CNN
 F 3 "" H 3150 3425 60  0000 C CNN
@@
 F 0 "D3" V 3875 4475 50  0000 R CNB
 F 1 "B220A-13-F" H 3925 4550 30  0000 R CNN
-F 2 "veloce:D_SMB" V 3800 4475 50  0001 C CNN
+F 2 "veloce:D_SMA" V 3800 4475 50  0001 C CNN
 F 3 "~" V 3800 4475 50  0001 C CNN
 	1    3800 4475
@@
 AR Path="/6276F530/627E9CF5" Ref="Q6"  Part="1"
 F 0 "Q6" H 3275 5300 50  0000 L CNB
-F 1 "RYM002N05" V 3350 4900 30  0000 L CNN
+F 1 "RUM001L02T2CL" V 3350 4900 30  0000 L CNN
 F 2 "veloce:SOT-723" H 3350 5125 29  0001 L CNN
 F 3 "" H 3150 5175 60  0000 C CNN
@@
 F 0 "D4" V 3875 6225 50  0000 R CNB
 F 1 "B220A-13-F" H 3925 6300 30  0000 R CNN
-F 2 "veloce:D_SMB" V 3800 6225 50  0001 C CNN
+F 2 "veloce:D_SMA" V 3800 6225 50  0001 C CNN
 F 3 "~" V 3800 6225 50  0001 C CNN
 	1    3800 6225
@@
 AR Path="/6276F530/627E9D48" Ref="Q8"  Part="1"
 F 0 "Q8" H 3275 7050 50  0000 L CNB
-F 1 "RYM002N05" V 3350 6650 30  0000 L CNN
+F 1 "RUM001L02T2CL" V 3350 6650 30  0000 L CNN
 F 2 "veloce:SOT-723" H 3350 6875 29  0001 L CNN
 F 3 "" H 3150 6925 60  0000 C CNN
@@
 F 0 "D5" V 6125 975 50  0000 R CNB
 F 1 "B220A-13-F" H 6175 1050 30  0000 R CNN
-F 2 "veloce:D_SMB" V 6050 975 50  0001 C CNN
+F 2 "veloce:D_SMA" V 6050 975 50  0001 C CNN
 F 3 "~" V 6050 975 50  0001 C CNN
 	1    6050 975
@@
 AR Path="/6276F530/627E9D9A" Ref="Q10"  Part="1"
 F 0 "Q10" H 5525 1800 50  0000 L CNB
-F 1 "RYM002N05" V 5600 1400 30  0000 L CNN
+F 1 "RUM001L02T2CL" V 5600 1400 30  0000 L CNN
 F 2 "veloce:SOT-723" H 5600 1625 29  0001 L CNN
 F 3 "" H 5400 1675 60  0000 C CNN
@@
 F 0 "D7" V 6125 4475 50  0000 R CNB
 F 1 "B220A-13-F" H 6175 4550 30  0000 R CNN
-F 2 "veloce:D_SMB" V 6050 4475 50  0001 C CNN
+F 2 "veloce:D_SMA" V 6050 4475 50  0001 C CNN
 F 3 "~" V 6050 4475 50  0001 C CNN
 	1    6050 4475
@@
 AR Path="/6276F530/627E9DED" Ref="Q14"  Part="1"
 F 0 "Q14" H 5525 5300 50  0000 L CNB
-F 1 "RYM002N05" V 5600 4900 30  0000 L CNN
+F 1 "RUM001L02T2CL" V 5600 4900 30  0000 L CNN
 F 2 "veloce:SOT-723" H 5600 5125 29  0001 L CNN
 F 3 "" H 5400 5175 60  0000 C CNN
@@
 F 0 "D6" V 6125 2725 50  0000 R CNB
 F 1 "B220A-13-F" H 6175 2800 30  0000 R CNN
-F 2 "veloce:D_SMB" V 6050 2725 50  0001 C CNN
+F 2 "veloce:D_SMA" V 6050 2725 50  0001 C CNN
 F 3 "~" V 6050 2725 50  0001 C CNN
 	1    6050 2725
@@
 AR Path="/6276F530/627E9E40" Ref="Q12"  Part="1"
 F 0 "Q12" H 5525 3550 50  0000 L CNB
-F 1 "RYM002N05" V 5600 3150 30  0000 L CNN
+F 1 "RUM001L02T2CL" V 5600 3150 30  0000 L CNN
 F 2 "veloce:SOT-723" H 5600 3375 29  0001 L CNN
 F 3 "" H 5400 3425 60  0000 C CNN
@@
 F 0 "D8" V 6125 6225 50  0000 R CNB
 F 1 "B220A-13-F" H 6175 6300 30  0000 R CNN
-F 2 "veloce:D_SMB" V 6050 6225 50  0001 C CNN
+F 2 "veloce:D_SMA" V 6050 6225 50  0001 C CNN
 F 3 "~" V 6050 6225 50  0001 C CNN
 	1    6050 6225
@@
 AR Path="/6276F530/627E9E93" Ref="Q16"  Part="1"
 F 0 "Q16" H 5525 7050 50  0000 L CNB
-F 1 "RYM002N05" V 5600 6650 30  0000 L CNN
+F 1 "RUM001L02T2CL" V 5600 6650 30  0000 L CNN
 F 2 "veloce:SOT-723" H 5600 6875 29  0001 L CNN
 F 3 "" H 5400 6925 60  0000 C CNN
