File: kicad_v2/veloce.kicad_pcb (KiCad board)
At the start: 2 copper layers, 116 x 105 mm, 146 parts, among them J1 OUT, J17 USB_A_stacked, J2 OUT, J20 Inputs, J3 OUT, J4 OUT, J5 OUT, J6 OUT, J7 OUT, J8 OUT, J9 PWR, P1 CONN_1, P2 CONN_1, P3 CONN_1, P4 CONN_1, P5 CONN_1, P6 CONN_1, P7 CONN_1, P8 CONN_1, P9 CONN_1, Q1 FQD11P06TM, Q10 RYM002N05, Q11 ZXMP7A17K, Q12 RYM002N05, Q13 ZXMP7A17K, Q14 RYM002N05, Q15 ZXMP7A17K, Q16 RYM002N05, Q2 RYM002N05, Q3 FQD11P06TM, Q4 RYM002N05, Q5 ZXMP7A17K, Q6 RYM002N05, Q7 ZXMP7A17K, Q8 RYM002N05, Q9 ZXMP7A17K, U1 Adafruit_HUZZAH_ESP32_breakou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

Commit message: CV rev2 PCB
Parts:
- added P10: CONN_1, veloce:TestPoint_THTPad_D3.0mm_Drill1.5mm, F.Cu at (107.5, 125.5)
- added P11: CONN_1, veloce:TestPoint_THTPad_D3.0mm_Drill1.5mm, F.Cu at (89.5, 125.5)
- added P12: CONN_1, veloce:TestPoint_THTPad_D3.0mm_Drill1.5mm, F.Cu at (94.5, 125.5)
- added P13: CONN_1, veloce:TestPoint_THTPad_D3.0mm_Drill1.5mm, F.Cu at (112.5, 125.5)
- added P14: CONN_1, veloce:TestPoint_THTPad_D3.0mm_Drill1.5mm, F.Cu at (102.5, 125.5)
- added kibuzzard-61BC3C42: G***, veloce:label_buck_input, F.Cu at (126.7, 136.3)
- added kibuzzard-61BC3C7D: G***, veloce:label_buck_output, F.Cu at (126.7, 96.3)
- added kibuzzard-61BC4209: G***, veloce:label_GND, F.Cu at (101.0, 122.5)
- added kibuzzard-61BC4209: G***, veloce:label_GND, F.Cu at (120.1, 151.1)
- added kibuzzard-61BC84E3: G***, veloce:label_5V_USB, F.Cu at (131.9, 49.2)
- G1: footprint veloce:VR_logo4 -> veloce:logo_CV_v2_silk2
- G2: footprint veloce:VR_logo5 -> veloce:VR_v2_mask_logo7
- G3: value Logo_Veloce -> LOGO; footprint veloce:VR_logo2 -> veloce:logo_VR_v2_mask
- G4: value Logo_Veloce -> LOGO; footprint veloce:VR_logo3 -> veloce:logo_CV_v2_silk
- moved G7 34.2 mm to (105.5, 80.0)
- moved G3 27.2 mm to (70.0, 113.0)
- moved G4 27.2 mm to (70.0, 113.0)
- moved G8 21.8 mm to (119.9, 120.5)
- moved G9 21.8 mm to (119.9, 120.5)
- moved G5 15.5 mm to (122.4, 107.6)
- moved G6 15.5 mm to (122.4, 107.6)
Routing:
- net /GND: track 969.4 -> 976.6 mm
- net /5V: track 162.6 -> 169.4 mm
- net /OUT8: track 59.4 -> 58.4 mm
- net /OUT3: track 20.4 -> 21.1 mm

Commit message: JLCpcb production files ready for CV rev 2
Parts:
- D1, D2, D3, D4, D5, D6, D7, D8: footprint veloce:D_SMB -> veloce:D_SMA
- G1: footprint veloce:logo_CV_v2_silk2 -> veloce:logo_CV_v2_silk; moved to B.Cu
- G2: footprint veloce:VR_v2_mask_logo7 -> veloce:logo_VR_v2_mask; moved to B.Cu
- G3: value LOGO -> Logo_Veloce; footprint veloce:logo_VR_v2_mask -> veloce:logo_CV_v2_silk2; moved to F.Cu
- G4: value LOGO -> Logo_Veloce; footprint veloce:logo_CV_v2_silk -> veloce:logo_CV_v2_mask2; moved to F.Cu
- Q10, Q12, Q14, Q16, Q2, Q4, Q6, Q8: value RYM002N05 -> RUM001L02T2CL
- R46: value 620E -> 510E
- R47: value 2k -> 1k8
- R48: value 7k5 -> 5k6
- moved G5 39.8 mm to (105.4, 71.6)
- moved G6 39.8 mm to (105.4, 71.6)
- moved G8 37.7 mm to (105.9, 85.5)
- moved G9 37.7 mm to (105.9, 85.5)
- moved G1 33.0 mm to (71.0, 111.0), turned to 180 degrees
- moved G2 33.0 mm to (71.0, 111.0), turned to 180 degrees
- moved G3 32.1 mm to (102.0, 110.0), turned to 0 degrees
- moved G4 32.1 mm to (102.0, 110.0), turned to 0 degrees
- moved G7 25.0 mm to (105.5, 55.0)
Routing:
- net /GND: track 976.6 -> 978.7 mm
