File: kicad_v2/veloce.sch (KiCad schematic (older format))
At the start: 51 parts, among them J17 USB_A_stacked, J20 Inputs, J9 PWR, P1 CONN_1, P2 CONN_1, P3 CONN_1, P4 CONN_1, P5 CONN_1, P6 CONN_1, P7 CONN_1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

Commit message: CV rev2 PCB
Parts:
- added P10, P11, P12, P13, P14: CONN_1, veloce:TestPoint_THTPad_D3.0mm_Drill1.5mm, symbol veloce:CONN_1
Connections:
- net GND: now also P10.1, P11.1, P12.1, P13.1, P14.1
Changed lines of the file:
@@
 	3725 2100 3325 2100
 Wire Wire Line
-	3725 2100 4125 2100
+	3725 2100 3925 2100
 Wire Wire Line
 	4525 2100 4525 2000
@@
 Connection ~ 4125 2100
 Wire Wire Line
-	4125 2100 4525 2100
+	4125 2100 4325 2100
 Wire Wire Line
 	3725 1350 3725 1300
@@
 Text Label 1675 2175 2    40   ~ 0
 GND
+$Comp
+L veloce:CONN_1 P10
+U 1 1 61BF2826
+P 3725 2250
+F 0 "P10" V 3775 2275 40  0000 R CNN
+F 1 "CONN_1" H 3725 2305 30  0001 C CNN
+F 2 "veloce:TestPoint_THTPad_D3.0mm_Drill1.5mm" H 3725 2250 60  0001 C CNN
+F 3 "" H 3725 2250 60  0000 C CNN
+	1    3725 2250
+	0    1    1    0
+$EndComp
+$Comp
+L veloce:CONN_1 P12
+U 1 1 61BF3CDC
+P 4125 2250
+F 0 "P12" V 4175 2275 40  0000 R CNN
+F 1 "CONN_1" H 4125 2305 30  0001 C CNN
+F 2 "veloce:TestPoint_THTPad_D3.0mm_Drill1.5mm" H 4125 2250 60  0001 C CNN
+F 3 "" H 4125 2250 60  0000 C CNN
+	1    4125 2250
+	0    1    1    0
+$EndComp
+$Comp
+L veloce:CONN_1 P14
+U 1 1 61BF4577
+P 4525 2250
+F 0 "P14" V 4575 2275 40  0000 R CNN
+F 1 "CONN_1" H 4525 2305 30  0001 C CNN
+F 2 "veloce:TestPoint_THTPad_D3.0mm_Drill1.5mm" H 4525 2250 60  0001 C CNN
+F 3 "" H 4525 2250 60  0000 C CNN
+	1    4525 2250
+	0    1    1    0
+$EndComp
+Connection ~ 4525 2100
+$Comp
+L veloce:CONN_1 P13
+U 1 1 61BF4C3F
+P 4325 2250
+F 0 "P13" V 4375 2275 40  0000 R CNN
+F 1 "CONN_1" H 4325 2305 30  0001 C CNN
+F 2 "veloce:TestPoint_THTPad_D3.0mm_Drill1.5mm" H 4325 2250 60  0001 C CNN
+F 3 "" H 4325 2250 60  0000 C CNN
+	1    4325 2250
+	0    1    1    0
+$EndComp
+Connection ~ 4325 2100
+Wire Wire Line
+	4325 2100 4525 2100
+$Comp
+L veloce:CONN_1 P11
+U 1 1 61BF51C8
+P 3925 2250
+F 0 "P11" V 3975 2275 40  0000 R CNN
+F 1 "CONN_1" H 3925 2305 30  0001 C CNN
+F 2 "veloce:TestPoint_THTPad_D3.0mm_Drill1.5mm" H 3925 2250 60  0001 C CNN
+F 3 "" H 3925 2250 60  0000 C CNN
+	1    3925 2250
+	0    1    1    0
+$EndComp
+Connection ~ 3925 2100
+Wire Wire Line
+	3925 2100 4125 2100
 $EndSCHEMATC

Commit message: JLCpcb production files ready for CV rev 2
Parts:
- G1: footprint veloce:VR_logo4 -> veloce:logo_CV_v2_silk
- G2: footprint veloce:VR_logo5 -> veloce:logo_VR_v2_mask
- G3: footprint veloce:VR_logo2 -> veloce:logo_CV_v2_silk2
- G4: footprint veloce:VR_logo3 -> veloce:logo_CV_v2_mask2
- R46: value 620E -> 510E
- R47: value 2k -> 1k8
- R48: value 7k5 -> 5k6
Changed lines of the file:
@@
 L veloce:Logo_Veloce G2
 U 1 1 6157474A
-P 8975 6850
-F 0 "G2" H 8975 6525 60  0001 C CNN
-F 1 "Logo_Veloce" H 8975 7175 60  0001 C CNN
-F 2 "veloce:VR_logo5" H 8975 6850 50  0001 C CNN
-F 3 "" H 8975 6850 50  0001 C CNN
-	1    8975 6850
+P 9350 6850
+F 0 "G2" H 9350 6525 60  0001 C CNN
+F 1 "Logo_Veloce" H 9350 7175 60  0001 C CNN
+F 2 "veloce:logo_VR_v2_mask" H 9350 6850 50  0001 C CNN
+F 3 "" H 9350 6850 50  0001 C CNN
+	1    9350 6850
 	1    0    0    -1
 $EndComp
@@
 L veloce:Logo_Veloce G3
 U 1 1 61576B43
-P 8975 6850
-F 0 "G3" H 8975 6525 60  0001 C CNN
-F 1 "Logo_Veloce" H 8975 7175 60  0001 C CNN
-F 2 "veloce:VR_logo2" H 8975 6850 50  0001 C CNN
-F 3 "" H 8975 6850 50  0001 C CNN
-	1    8975 6850
+P 9875 6850
+F 0 "G3" H 9875 6525 60  0001 C CNN
+F 1 "Logo_Veloce" H 9875 7175 60  0001 C CNN
+F 2 "veloce:logo_CV_v2_silk2" H 9875 6850 50  0001 C CNN
+F 3 "" H 9875 6850 50  0001 C CNN
+	1    9875 6850
 	1    0    0    -1
 $EndComp
@@
 L veloce:Logo_Veloce G4
 U 1 1 61579302
-P 8975 6850
-F 0 "G4" H 8975 6525 60  0001 C CNN
-F 1 "Logo_Veloce" H 8975 7175 60  0001 C CNN
-F 2 "veloce:VR_logo3" H 8975 6850 50  0001 C CNN
-F 3 "" H 8975 6850 50  0001 C CNN
-	1    8975 6850
+P 10425 6850
+F 0 "G4" H 10425 6525 60  0001 C CNN
+F 1 "Logo_Veloce" H 10425 7175 60  0001 C CNN
+F 2 "veloce:logo_CV_v2_mask2" H 10425 6850 50  0001 C CNN
+F 3 "" H 10425 6850 50  0001 C CNN
+	1    10425 6850
 	1    0    0    -1
 $EndComp
@@
 L veloce:Logo_Veloce G1
 U 1 1 6157F0FB
-P 8975 6850
-F 0 "G1" H 8975 6525 60  0001 C CNN
-F 1 "Logo_Veloce" H 8975 7175 60  0001 C CNN
-F 2 "veloce:VR_logo4" H 8975 6850 50  0001 C CNN
-F 3 "" H 8975 6850 50  0001 C CNN
-	1    8975 6850
+P 8800 6850
+F 0 "G1" H 8800 6525 60  0001 C CNN
+F 1 "Logo_Veloce" H 8800 7175 60  0001 C CNN
+F 2 "veloce:logo_CV_v2_silk" H 8800 6850 50  0001 C CNN
+F 3 "" H 8800 6850 50  0001 C CNN
+	1    8800 6850
 	1    0    0    -1
 $EndComp
@@
 P 3725 1500
 F 0 "R46" H 3800 1550 50  0000 L CNN
-F 1 "620E" V 3725 1425 40  0000 L CNN
+F 1 "510E" V 3725 1425 40  0000 L CNN
 F 2 "veloce:R_0805_2012Metric" V 3655 1500 50  0001 C CNN
 F 3 "~" H 3725 1500 50  0001 C CNN
@@
 P 4525 1500
 F 0 "R48" H 4600 1550 50  0000 L CNN
-F 1 "7k5" V 4525 1425 40  0000 L CNN
+F 1 "5k6" V 4525 1425 40  0000 L CNN
 F 2 "veloce:R_0805_2012Metric" V 4455 1500 50  0001 C CNN
 F 3 "~" H 4525 1500 50  0001 C CNN
@@
 P 4125 1500
 F 0 "R47" H 4200 1550 50  0000 L CNN
-F 1 "2k" V 4125 1425 40  0000 L CNN
+F 1 "1k8" V 4125 1425 40  0000 L CNN
 F 2 "veloce:R_0805_2012Metric" V 4055 1500 50  0001 C CNN
 F 3 "~" H 4125 1500 50  0001 C CNN
